Commit message: 硬件组件内部添加重力补偿

File: robot_config/config/robot_1.ros2_control.xacro (robot description, xacro)
@@ -6,8 +6,10 @@
             <hardware>
                 <!-- By default, set up controllers for simulation. This won't work on real hardware -->
-                <!-- <plugin>mobile_base_hardware/MobileBaseHardwareInterface</plugin> -->
-                <plugin>mock_components/GenericSystem</plugin>
+                <plugin>mobile_base_hardware/MobileBaseHardwareInterface</plugin>
+                <!-- <plugin>mock_components/GenericSystem</plugin> -->
             </hardware>
             <joint name="joint_1">
+                <param name="kp">80.0</param>
+                <param name="kd">10.0</param>
                 <command_interface name="position"/>
                 <state_interface name="position">
@@ -17,4 +19,6 @@
             </joint>
             <joint name="joint_2">
+                <param name="kp">90.0</param>
+                <param name="kd">15.0</param>
                 <command_interface name="position"/>
                 <state_interface name="position">
@@ -24,4 +28,6 @@
             </joint>
             <joint name="joint_3">
+                <param name="kp">100.0</param>
+                <param name="kd">15.0</param>
                 <command_interface name="position"/>
                 <state_interface name="position">
@@ -31,4 +37,6 @@
             </joint>
             <joint name="joint_4">
+                <param name="kp">20.0</param>
+                <param name="kd">1.0</param>
                 <command_interface name="position"/>
                 <state_interface name="position">
@@ -38,4 +46,6 @@
             </joint>
             <joint name="joint_5">
+                <param name="kp">20.0</param>
+                <param name="kd">1.0</param>
                 <command_interface name="position"/>
                 <state_interface name="position">
@@ -45,4 +55,6 @@
             </joint>
             <joint name="joint_6">
+                <param name="kp">10.0</param>
+                <param name="kd">1.0</param>
                 <command_interface name="position"/>
                 <state_interface name="position">

File: robot_description/urdf/robot_1.urdf (robot description, URDF)
Before this commit: robot robot_1, 7 links, 6 joints
Links:
- link base_link: mass 1.4290004 -> 4.06800157701675
- link link_1: mass 0.8693372 -> 0.6895799
- link link_2: mass 0.7057861 -> 0.6370289
- link link_3: mass 0.7424189 -> 0.7024189
- link link_4: mass 0.6182432 -> 0.5211502
- link link_5: mass 0.5144253 -> 0.4734144
Joints:
- joint joint_1: limit lower=-3 upper=3 effort=7 velocity=3 -> lower=-3 upper=3 effort=27 velocity=3; origin xyz=0 0 0.0995 rpy=0 0 0 -> xyz=0.00019927 -0.001877 0.10675 rpy=0 0 0
- joint joint_3: origin xyz=-0.1798 0 -0.00087243 rpy=-3.1416 0 0 -> xyz=-0.18 0 0 rpy=-3.1416 0 0
- joint joint_4: limit lower=-3.13 upper=3.13 effort=27 velocity=3 -> lower=-3 upper=3 effort=7 velocity=3; origin xyz=0.0029242 0.071801 -0.00087243 rpy=1.5708 0 1.5708 -> xyz=-0.00071398 0.071768 -0.00087296 rpy=1.5708 0 1.5708
- joint joint_5: axis 0 0 1 -> 0 0 -1; limit lower=-1.57 upper=1.57 effort=7 velocity=3 -> lower=-3 upper=3 effort=7 velocity=3; origin xyz=0.00019933 0.004294 0.20686 rpy=-1.5708 0 0 -> xyz=0.00023228 -0.0022353 0.20325 rpy=-1.5708 0 0
- joint joint_6: origin xyz=0.00023228 -0.061253 -0.00048535 rpy=1.5708 0 0 -> xyz=-0.00023228 -0.061253 0.0014853 rpy=1.5708 0 0
